File: Hardware/Hoerbaer/audio.kicad_sch (KiCad schematic)
At the start: 37 parts, among them J14 Speaker_L, J15 Speaker_R, U10 TAS5805M

Commit message: Order numbers
Parts:
- C33, C46, C47, C48, C49, C51, C52, C53, C54: JLCPCB (none) -> C267415; MPN (none) -> C1005X7R222MGTS
- C36, C43, C50: JLCPCB (none) -> C458949; MPN (none) -> MT15B104K160CT
- C39, C40, C41, C42: JLCPCB (none) -> C915854; MPN (none) -> TCC0402X7R224K250AT
- U10: JLCPCB (none) -> C478472; MPN (none) -> TAS5805MPWPR
Changed lines of the file:
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@@
+      (effects (font (size 1.27 1.27)) hide)
+    )
+    (property "JLCPCB" "C267415" (at 214.63 121.92 0)
+      (effects (font (size 1.27 1.27)) hide)
+    )
+    (property "MPN" "C1005X7R222MGTS" (at 214.63 121.92 0)
       (effects (font (size 1.27 1.27)) hide)
     )
@@
       (effects (font (size 1.27 1.27)) hide)
     )
+    (property "JLCPCB" "C267415" (at 228.6 90.17 0)
+      (effects (font (size 1.27 1.27)) hide)
+    )
+    (property "MPN" "C1005X7R222MGTS" (at 228.6 90.17 0)
+      (effects (font (size 1.27 1.27)) hide)
+    )
     (pin "1")
     (pin "2")
@@
       (effects (font (size 1.27 1.27)) hide)
     )
+    (property "JLCPCB" "C267415" (at 33.02 45.72 0)
+      (effects (font (size 1.27 1.27)) hide)
+    )
+    (property "MPN" "C1005X7R222MGTS" (at 33.02 45.72 0)
+      (effects (font (size 1.27 1.27)) hide)
+    )
     (pin "1")
     (pin "2")
@@
       (effects (font (size 1.27 1.27)) hide)
     )
+    (property "JLCPCB" "C915854" (at 175.26 100.33 0)
+      (effects (font (size 1.27 1.27)) hide)
+    )
+    (property "MPN" "TCC0402X7R224K250AT" (at 175.26 100.33 0)
+      (effects (font (size 1.27 1.27)) hide)
+    )
     (pin "1")
     (pin "2")
@@
       (effects (font (size 1.27 1.27)) hide)
     )
+    (property "JLCPCB" "C267415" (at 228.6 74.93 0)
+      (effects (font (size 1.27 1.27)) hide)
+    )
+    (property "MPN" "C1005X7R222MGTS" (at 228.6 74.93 0)
+      (effects (font (size 1.27 1.27)) hide)
+    )
     (pin "1")
     (pin "2")
@@
       (effects (font (size 1.27 1.27)) hide)
     )
+    (property "JLCPCB" "C267415" (at 214.63 90.17 0)
+      (effects (font (size 1.27 1.27)) hide)
+    )
+    (property "MPN" "C1005X7R222MGTS" (at 214.63 90.17 0)
+      (effects (font (size 1.27 1.27)) hide)
+    )
     (pin "1")
     (pin "2")
@@
       (effects (font (size 1.27 1.27)) hide)
     )
+    (property "JLCPCB" "C267415" (at 228.6 106.68 0)
+      (effects (font (size 1.27 1.27)) hide)
+    )
+    (property "MPN" "C1005X7R222MGTS" (at 228.6 106.68 0)
+      (effects (font (size 1.27 1.27)) hide)
+    )
     (pin "1")
     (pin "2")
@@
       (effects (font (size 1.27 1.27)) hide)
     )
+    (property "JLCPCB" "C915854" (at 175.26 114.3 0)
+      (effects (font (size 1.27 1.27)) hide)
+    )
+    (property "MPN" "TCC0402X7R224K250AT" (at 175.26 114.3 0)
+      (effects (font (size 1.27 1.27)) hide)
+    )
     (pin "1")
     (pin "2")
@@
       (effects (font (size 1.27 1.27)) hide)
     )
+    (property "JLCPCB" "C915854" (at 175.26 77.47 0)
+      (effects (font (size 1.27 1.27)) hide)
+    )
+    (property "MPN" "TCC0402X7R224K250AT" (at 175.26 77.47 0)
+      (effects (font (size 1.27 1.27)) hide)
+    )
     (pin "1")
     (pin "2")
@@
       (effects (font (size 1.27 1.27)) hide)
     )
+    (property "JLCPCB" "C458949" (at 228.6 39.37 0)
+      (effects (font (size 1.27 1.27)) hide)
+    )
+    (property "MPN" "MT15B104K160CT" (at 228.6 39.37 0)
+      (effects (font (size 1.27 1.27)) hide)
+    )
     (pin "1")
     (pin "2")
@@
       (effects (font (size 1.27 1.27)) hide)
     )
+    (property "JLCPCB" "C267415" (at 214.63 106.68 0)
+      (effects (font (size 1.27 1.27)) hide)
+    )
+    (property "MPN" "C1005X7R222MGTS" (at 214.63 106.68 0)
+      (effects (font (size 1.27 1.27)) hide)
+    )
     (pin "1")
     (pin "2")
@@
     )
     (property "Datasheet" "~" (at 175.26 91.44 0)
+      (effects (font (size 1.27 1.27)) hide)
+    )
+    (property "JLCPCB" "C915854" (at 175.26 91.44 0)
+      (effects (font (size 1.27 1.27)) hide)
+    )
+    (property "MPN" "TCC0402X7R224K250AT" (at 175.26 91.44 0)
       (effects (font (size 1.27 1.27)) hide)
     )
@@
       (effects (font (size 1.27 1.27)) hide)
     )
+    (property "JLCPCB" "C458949" (at 107.95 39.37 0)
+      (effects (font (size 1.27 1.27)) hide)
+    )
+    (property "MPN" "MT15B104K160CT" (at 107.95 39.37 0)
+      (effects (font (size 1.27 1.27)) hide)
+    )
     (pin "1")
     (pin "2")
@@
       (effects (font (size 1.27 1.27)) hide)
     )
+    (property "JLCPCB" "C267415" (at 214.63 74.93 0)
+      (effects (font (size 1.27 1.27)) hide)
+    )
+    (property "MPN" "C1005X7R222MGTS" (at 214.63 74.93 0)
+      (effects (font (size 1.27 1.27)) hide)
+    )
     (pin "1")
     (pin "2")
@@
     )
     (property "Datasheet" "~" (at 166.37 39.37 0)
+      (effects (font (size 1.27 1.27)) hide)
+    )
+    (property "JLCPCB" "C458949" (at 166.37 39.37 0)
+      (effects (font (size 1.27 1.27)) hide)
+    )
+    (property "MPN" "MT15B104K160CT" (at 166.37 39.37 0)
       (effects (font (size 1.27 1.27)) hide)
     )
@@
     )
     (property "Datasheet" "https://www.ti.com/lit/gpn/tas5805m" (at 147.32 142.24 0)
+      (effects (font (size 1.27 1.27)) hide)
+    )
+    (property "JLCPCB" "C478472" (at 147.32 96.52 0)
+      (effects (font (size 1.27 1.27)) hide)
+    )
+    (property "MPN" "TAS5805MPWPR" (at 147.32 96.52 0)
       (effects (font (size 1.27 1.27)) hide)
     )
@@
       (effects (font (size 1.27 1.27)) hide)
     )
+    (property "JLCPCB" "C267415" (at 228.6 121.92 0)
+      (effects (font (size 1.27 1.27)) hide)
+    )
+    (property "MPN" "C1005X7R222MGTS" (at 228.6 121.92 0)
+      (effects (font (size 1.27 1.27)) hide)
+    )

Commit message: Renamed JLCPCB attribute to LCSC (plugin search list)
Parts:
- C33, C46, C47, C48, C49, C51, C52, C53, C54: JLCPCB C267415 -> (none); LCSC (none) -> C267415
- C34, C35: JLCPCB C726581 -> (none); LCSC (none) -> C726581
- C36, C43, C50: JLCPCB C458949 -> (none); LCSC (none) -> C458949
- C37, C38, C44, C45: JLCPCB C6120032 -> (none); LCSC (none) -> C6120032
- C39, C40, C41, C42: JLCPCB C915854 -> (none); LCSC (none) -> C915854
- C55: JLCPCB C361188 -> (none); LCSC (none) -> C361188
- FB1: JLCPCB C316421 -> (none); LCSC (none) -> C316421
- FB2, FB3, FB4, FB5: JLCPCB C370090 -> (none); LCSC (none) -> C370090
- U10: JLCPCB C478472 -> (none); LCSC (none) -> C478472
Changed lines of the file:
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@@
       (effects (font (size 1.27 1.27)) hide)
     )
-    (property "JLCPCB" "C726581" (at 113.03 74.93 0)
+    (property "LCSC" "C726581" (at 113.03 74.93 0)
       (effects (font (size 1.27 1.27)) hide)
     )
@@
       (effects (font (size 1.27 1.27)) hide)
     )
-    (property "JLCPCB" "C267415" (at 214.63 121.92 0)
+    (property "LCSC" "C267415" (at 214.63 121.92 0)
       (effects (font (size 1.27 1.27)) hide)
     )
@@
       (effects (font (size 1.27 1.27)) hide)
     )
-    (property "JLCPCB" "C726581" (at 118.11 77.47 0)
+    (property "LCSC" "C726581" (at 118.11 77.47 0)
       (effects (font (size 1.27 1.27)) hide)
     )
@@
       (effects (font (size 1.27 1.27)) hide)
     )
-    (property "JLCPCB" "C267415" (at 228.6 90.17 0)
+    (property "LCSC" "C267415" (at 228.6 90.17 0)
       (effects (font (size 1.27 1.27)) hide)
     )
@@
       (effects (font (size 1.27 1.27)) hide)
     )
-    (property "JLCPCB" "C267415" (at 33.02 45.72 0)
+    (property "LCSC" "C267415" (at 33.02 45.72 0)
       (effects (font (size 1.27 1.27)) hide)
     )
@@
       (effects (font (size 1.27 1.27)) hide)
     )
-    (property "JLCPCB" "C915854" (at 175.26 100.33 0)
+    (property "LCSC" "C915854" (at 175.26 100.33 0)
       (effects (font (size 1.27 1.27)) hide)
     )
@@
       (effects (font (size 1.27 1.27)) hide)
     )
-    (property "JLCPCB" "C6120032" (at 140.97 39.37 0)
+    (property "LCSC" "C6120032" (at 140.97 39.37 0)
       (effects (font (size 1.27 1.27)) hide)
     )
@@
       (effects (font (size 1.27 1.27)) hide)
     )
-    (property "JLCPCB" "C361188" (at 240.03 39.37 0)
+    (property "LCSC" "C361188" (at 240.03 39.37 0)
       (effects (font (size 1.27 1.27)) hide)
     )
@@
       (effects (font (size 1.27 1.27)) hide)
     )
-    (property "JLCPCB" "C267415" (at 228.6 74.93 0)
+    (property "LCSC" "C267415" (at 228.6 74.93 0)
       (effects (font (size 1.27 1.27)) hide)
     )
@@
       (effects (font (size 1.27 1.27)) hide)
     )
-    (property "JLCPCB" "C267415" (at 214.63 90.17 0)
+    (property "LCSC" "C267415" (at 214.63 90.17 0)
       (effects (font (size 1.27 1.27)) hide)
     )
@@
       (effects (font (size 1.27 1.27)) hide)
     )
-    (property "JLCPCB" "C267415" (at 228.6 106.68 0)
+    (property "LCSC" "C267415" (at 228.6 106.68 0)
       (effects (font (size 1.27 1.27)) hide)
     )
@@
       (effects (font (size 1.27 1.27)) hide)
     )
-    (property "JLCPCB" "C915854" (at 175.26 114.3 0)
+    (property "LCSC" "C915854" (at 175.26 114.3 0)
       (effects (font (size 1.27 1.27)) hide)
     )
@@
       (effects (font (size 1.27 1.27)) hide)
     )
-    (property "JLCPCB" "C915854" (at 175.26 77.47 0)
+    (property "LCSC" "C915854" (at 175.26 77.47 0)
       (effects (font (size 1.27 1.27)) hide)
     )
@@
       (effects (font (size 1.27 1.27)) hide)
     )
-    (property "JLCPCB" "C458949" (at 228.6 39.37 0)
+    (property "LCSC" "C458949" (at 228.6 39.37 0)
       (effects (font (size 1.27 1.27)) hide)
     )
@@
       (effects (font (size 1.27 1.27)) hide)
     )
-    (property "JLCPCB" "C316421" (at 44.45 40.64 90)
+    (property "LCSC" "C316421" (at 44.45 40.64 90)
       (effects (font (size 1.27 1.27)) hide)
     )
@@
       (effects (font (size 1.27 1.27)) hide)
     )
-    (property "JLCPCB" "C370090" (at 208.28 119.38 90)
+    (property "LCSC" "C370090" (at 208.28 119.38 90)
       (effects (font (size 1.27 1.27)) hide)
     )
@@
       (effects (font (size 1.27 1.27)) hide)
     )
-    (property "JLCPCB" "C6120032" (at 199.39 39.37 0)
+    (property "LCSC" "C6120032" (at 199.39 39.37 0)
       (effects (font (size 1.27 1.27)) hide)
     )
@@
       (effects (font (size 1.27 1.27)) hide)
     )
-    (property "JLCPCB" "C6120032" (at 179.07 39.37 0)
+    (property "LCSC" "C6120032" (at 179.07 39.37 0)
       (effects (font (size 1.27 1.27)) hide)
     )
@@
       (effects (font (size 1.27 1.27)) hide)
     )
-    (property "JLCPCB" "C267415" (at 214.63 106.68 0)
+    (property "LCSC" "C267415" (at 214.63 106.68 0)
       (effects (font (size 1.27 1.27)) hide)
     )
@@
       (effects (font (size 1.27 1.27)) hide)
     )
-    (property "JLCPCB" "C915854" (at 175.26 91.44 0)
+    (property "LCSC" "C915854" (at 175.26 91.44 0)
       (effects (font (size 1.27 1.27)) hide)
     )
@@
       (effects (font (size 1.27 1.27)) hide)
     )
-    (property "JLCPCB" "C370090" (at 208.28 72.39 90)
+    (property "LCSC" "C370090" (at 208.28 72.39 90)
       (effects (font (size 1.27 1.27)) hide)
     )
@@
       (effects (font (size 1.27 1.27)) hide)
     )
-    (property "JLCPCB" "C458949" (at 107.95 39.37 0)
+    (property "LCSC" "C458949" (at 107.95 39.37 0)
       (effects (font (size 1.27 1.27)) hide)
     )
@@
       (effects (font (size 1.27 1.27)) hide)
     )
-    (property "JLCPCB" "C267415" (at 214.63 74.93 0)
+    (property "LCSC" "C267415" (at 214.63 74.93 0)
       (effects (font (size 1.27 1.27)) hide)
     )
@@
       (effects (font (size 1.27 1.27)) hide)
     )
-    (property "JLCPCB" "C458949" (at 166.37 39.37 0)
+    (property "LCSC" "C458949" (at 166.37 39.37 0)
       (effects (font (size 1.27 1.27)) hide)
     )
@@
       (effects (font (size 1.27 1.27)) hide)
     )
-    (property "JLCPCB" "C370090" (at 208.28 104.14 90)
+    (property "LCSC" "C370090" (at 208.28 104.14 90)
       (effects (font (size 1.27 1.27)) hide)
     )
@@
       (effects (font (size 1.27 1.27)) hide)
     )
-    (property "JLCPCB" "C478472" (at 147.32 96.52 0)
+    (property "LCSC" "C478472" (at 147.32 96.52 0)
       (effects (font (size 1.27 1.27)) hide)
     )
@@
       (effects (font (size 1.27 1.27)) hide)
     )
-    (property "JLCPCB" "C267415" (at 228.6 121.92 0)
+    (property "LCSC" "C267415" (at 228.6 121.92 0)
       (effects (font (size 1.27 1.27)) hide)
     )
@@
       (effects (font (size 1.27 1.27)) hide)
     )
-    (property "JLCPCB" "C6120032" (at 120.65 39.37 0)
+    (property "LCSC" "C6120032" (at 120.65 39.37 0)
       (effects (font (size 1.27 1.27)) hide)
     )
@@
       (effects (font (size 1.27 1.27)) hide)
     )
-    (property "JLCPCB" "C370090" (at 208.28 87.63 90)
-      (effects (font (size 1.27 1.27)) hide)
-    )
+    (property "LCSC" "C370090" (at 208.28 87.63 90)
+      (effects (font (size 1.27 1.27)) hide)
+    )

Commit message: Resistor Order Numbers
Parts:
- R61: LCSC (none) -> C25744; MPN (none) -> 0402WGF1002TCE
- R62: LCSC (none) -> C25900; MPN (none) -> 0402WGF4701TCE
- R63, R64, R65, R66: LCSC (none) -> C25131; MPN (none) -> 0402WGF680JTCE
Changed lines of the file:
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@@
+      (effects (font (size 1.27 1.27)) hide)
+    )
+    (property "LCSC" "C25131" (at 228.6 80.01 0)
+      (effects (font (size 1.27 1.27)) hide)
+    )
+    (property "MPN" "0402WGF680JTCE" (at 228.6 80.01 0)
       (effects (font (size 1.27 1.27)) hide)
     )
@@
       (effects (font (size 1.27 1.27)) hide)
     )
+    (property "LCSC" "C25900" (at 100.33 104.14 0)
+      (effects (font (size 1.27 1.27)) hide)
+    )
+    (property "MPN" "0402WGF4701TCE" (at 100.33 104.14 0)
+      (effects (font (size 1.27 1.27)) hide)
+    )
     (pin "1")
     (pin "2")
@@
       (effects (font (size 1.27 1.27)) hide)
     )
+    (property "LCSC" "C25131" (at 228.6 95.25 0)
+      (effects (font (size 1.27 1.27)) hide)
+    )
+    (property "MPN" "0402WGF680JTCE" (at 228.6 95.25 0)
+      (effects (font (size 1.27 1.27)) hide)
+    )
     (pin "1")
     (pin "2")
@@
       (effects (font (size 1.27 1.27)) hide)
     )
+    (property "LCSC" "C25744" (at 48.26 96.52 0)
+      (effects (font (size 1.27 1.27)) hide)
+    )
+    (property "MPN" "0402WGF1002TCE" (at 48.26 96.52 0)
+      (effects (font (size 1.27 1.27)) hide)
+    )
     (pin "1")
     (pin "2")
@@
       (effects (font (size 1.27 1.27)) hide)
     )
+    (property "LCSC" "C25131" (at 228.6 127 0)
+      (effects (font (size 1.27 1.27)) hide)
+    )
+    (property "MPN" "0402WGF680JTCE" (at 228.6 127 0)
+      (effects (font (size 1.27 1.27)) hide)
+    )
     (pin "1")
     (pin "2")
@@
       (effects (font (size 1.27 1.27)) hide)
     )
+    (property "LCSC" "C25131" (at 228.6 111.76 0)
+      (effects (font (size 1.27 1.27)) hide)
+    )
+    (property "MPN" "0402WGF680JTCE" (at 228.6 111.76 0)
+      (effects (font (size 1.27 1.27)) hide)
+    )
