File: Hardware/Hoerbaer/audio.kicad_sch (KiCad schematic)
At the start: 37 parts, among them J14 Speaker_L, J15 Speaker_R, U10 TAS5805M

Commit message: Fixed net tie ground plane issue.
Parts:
- U10: JLCPCB Rotation Offset (none) -> 90
Changed lines of the file:
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@@
+      (effects (font (size 1.27 1.27)) hide)
+    )
+    (property "JLCPCB Rotation Offset" "90" (at 147.32 96.52 0)
       (effects (font (size 1.27 1.27)) hide)
     )

Commit message: Many small corrections, changed connectors, ...
Parts:
- J14, J15: footprint Connector_Phoenix_MSTB:PhoenixContact_MSTBVA_2,5_2-G-5,08_1x02_P5.08mm_Vertical -> TerminalBlock:TerminalBlock_bornier-2_P5.08mm; LCSC (none) -> C8465; MPN (none) -> WJ500V-5.08-2P; now not fitted
Connections:
- net SPEAKER_A+: now also J14.2 (Pin_2); no longer J14.1 (Pin_1)
- net SPEAKER_A-: now also J14.1 (Pin_1); no longer J14.2 (Pin_2)
Changed lines of the file:
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@@
     )
   )
-  (symbol (lib_id "Connector_Generic:Conn_01x02") (at 245.11 85.09 0) (unit 1)
-    (in_bom yes) (on_board yes) (dnp no) (fields_autoplaced)
-    (property "Reference" "J14" (at 247.65 85.09 0)
-      (effects (font (size 1.27 1.27)) (justify left))
-    )
-    (property "Value" "Speaker_L" (at 247.65 87.63 0)
-      (effects (font (size 1.27 1.27)) (justify left))
-    )
-    (property "Footprint" "Connector_Phoenix_MSTB:PhoenixContact_MSTBVA_2,5_2-G-5,08_1x02_P5.08mm_Vertical" (at 245.11 85.09 0)
-      (effects (font (size 1.27 1.27)) hide)
-    )
-    (property "Datasheet" "~" (at 245.11 85.09 0)
+  (symbol (lib_id "Connector_Generic:Conn_01x02") (at 245.11 87.63 0) (mirror x) (unit 1)
+    (in_bom yes) (on_board yes) (dnp yes)
+    (property "Reference" "J14" (at 247.65 87.63 0)
+      (effects (font (size 1.27 1.27)) (justify left))
+    )
+    (property "Value" "Speaker_L" (at 247.65 85.09 0)
+      (effects (font (size 1.27 1.27)) (justify left))
+    )
+    (property "Footprint" "TerminalBlock:TerminalBlock_bornier-2_P5.08mm" (at 245.11 87.63 0)
+      (effects (font (size 1.27 1.27)) hide)
+    )
+    (property "Datasheet" "~" (at 245.11 87.63 0)
+      (effects (font (size 1.27 1.27)) hide)
+    )
+    (property "MPN" "WJ500V-5.08-2P" (at 245.11 87.63 0)
+      (effects (font (size 1.27 1.27)) hide)
+    )
+    (property "LCSC" "C8465" (at 245.11 87.63 0)
       (effects (font (size 1.27 1.27)) hide)
     )
@@
   )
   (symbol (lib_id "Connector_Generic:Conn_01x02") (at 245.11 104.14 0) (unit 1)
-    (in_bom yes) (on_board yes) (dnp no) (fields_autoplaced)
+    (in_bom yes) (on_board yes) (dnp yes) (fields_autoplaced)
     (property "Reference" "J15" (at 247.65 104.14 0)
       (effects (font (size 1.27 1.27)) (justify left))
@@
       (effects (font (size 1.27 1.27)) (justify left))
     )
-    (property "Footprint" "Connector_Phoenix_MSTB:PhoenixContact_MSTBVA_2,5_2-G-5,08_1x02_P5.08mm_Vertical" (at 245.11 104.14 0)
+    (property "Footprint" "TerminalBlock:TerminalBlock_bornier-2_P5.08mm" (at 245.11 104.14 0)
       (effects (font (size 1.27 1.27)) hide)
     )
@@
       (effects (font (size 1.27 1.27)) hide)
     )
+    (property "LCSC" "C8465" (at 245.11 104.14 0)
+      (effects (font (size 1.27 1.27)) hide)
+    )
+    (property "MPN" "WJ500V-5.08-2P" (at 245.11 104.14 0)
+      (effects (font (size 1.27 1.27)) hide)
+    )

Commit message: Fixed 1uF order number.
Parts:
- C34, C35: LCSC C726581 -> C29266; MPN AC0805KKX7R6BB105 -> CL05A105KO5NNNC
Changed lines of the file:
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@@
       (effects (font (size 1.27 1.27)) hide)
     )
-    (property "LCSC" "C726581" (at 113.03 74.93 0)
-      (effects (font (size 1.27 1.27)) hide)
-    )
-    (property "MPN" "AC0805KKX7R6BB105" (at 113.03 74.93 0)
+    (property "LCSC" "C29266 " (at 113.03 74.93 0)
+      (effects (font (size 1.27 1.27)) hide)
+    )
+    (property "MPN" "CL05A105KO5NNNC" (at 113.03 74.93 0)
       (effects (font (size 1.27 1.27)) hide)
     )
@@
       (effects (font (size 1.27 1.27)) hide)
     )
-    (property "LCSC" "C726581" (at 118.11 77.47 0)
-      (effects (font (size 1.27 1.27)) hide)
-    )
-    (property "MPN" "AC0805KKX7R6BB105" (at 118.11 77.47 0)
-      (effects (font (size 1.27 1.27)) hide)
-    )
+    (property "LCSC" "C29266 " (at 118.11 77.47 0)
+      (effects (font (size 1.27 1.27)) hide)
+    )
+    (property "MPN" "CL05A105KO5NNNC" (at 118.11 77.47 0)
+      (effects (font (size 1.27 1.27)) hide)
+    )

Commit message: WIP new hw rev
Parts:
- C42: renamed from C34; value 1µF, 10V -> 1µF, 16V; LCSC C29266 -> C29266
- C43: renamed from C35; value 1µF, 10V -> 1µF, 16V; LCSC C29266 -> C29266
- renumbered C33 to C40, C36 to C41, C37 to C44, C38 to C45, C43 to C46, C39 to C47, C40 to C48, C41 to C49, C42 to C50, C44 to C51, C45 to C52, C46 to C53, C47 to C54, C48 to C55, C49 to C56, C50 to C57, C51 to C58, C52 to C59, C53 to C60, C54 to C61, C55 to C62, J14 to J16, J15 to J17, R61 to R58, R62 to R59, R63 to R60, R64 to R61, R65 to R62, R66 to R63, U10 to U12
Connections:
- net VCC: no longer U12.2 (DVDD)
- net +12V renamed +9V
- new net VCC_P: U12.2 (DVDD)
Other:
- note added: "Inductor Variante https://jlcpcb.com/partdetail/Sumida-CDRH105RNP100NC/C171589"
- note added: "Input Filter (VHIGH => PVDD)"
- note removed: "Input Filter (VBAT => PVDD)"

Commit message: Layout, mono-jumpers
Parts:
- added JP11: MONO_B, Jumper:SolderJumper-3_P1.3mm_Bridged12_RoundedPad1.0x1.5mm, symbol Jumper:SolderJumper_3_Bridged12
- added JP12: MONO_A, Jumper:SolderJumper-3_P1.3mm_Bridged12_RoundedPad1.0x1.5mm, symbol Jumper:SolderJumper_3_Bridged12
Connections:
- net VCC is gone; now on net VCC_P: C57.1, C62.1, R59.1
- net AMP_OUT_A+: now also JP12.3 (B)
- net AMP_OUT_A-: now also JP12.2 (C); no longer FB3.1
- net AMP_OUT_B+: now also JP11.3 (B)
- net AMP_OUT_B-: now also JP11.2 (C); no longer FB5.1
- new net: FB5.1, JP11.1 (A)
- new net: FB3.1, JP12.1 (A)
Other:
- moved on the sheet: C53, C54, C55, C56, C58, C59, C60, C61, FB2, FB3, FB4, FB5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

Commit message: BOM FIxes
Parts:
- C40, C53, C54, C55, C56, C58, C59, C60, C61: LCSC C267415 -> C84703; MPN C1005X7R222MGTS -> CL05B222KB5NNNC
- C41, C46, C57: LCSC C458949 -> C1525; MPN MT15B104K160CT -> CL05B104KO5NNNC
Changed lines of the file:
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@@
 			"cykKCQkob25fYm9hcmQgeWVzKQoJCShkbnAgbm8pCgkJKHV1aWQgIjgxMzhiZTQ5LThkZmMtNDNi"
 			"Yy1iYjJhLTZhNjY0YjQzNzQ5NiIpCgkJKHByb3BlcnR5ICJSZWZlcmVuY2UiICIjUFdSMDQ3IgoJ"
-			"CQkoYXQgMjU3LjgxIDE0Ni4wNSAwKQoJCQkoZQ=="
+			"CQkoYXQgMjU3LjgxIDE0Ni4wNSAwKQoJCQkoZQAAAAAlBQAAAAAAALz/2wMAAAAAvJWpAwAAAAAm"
+			"BQAAAAAAAFr92wMAAAAAcXepAwAAAAAnBQAAAAAAACXT2wMAAAAA9myoAwAAAAAoBQAAAAAAADSU"
+			"3QMAAAAA9myoAwAAAAApBQAAAAAAAMV73gMAAAAAGHypAwAAAAAqBQAAAAAAAK9D7QMAAAAAGHyp"
+			"AwAAAAArBQAAAAAAADgm7gMAAAAAj5moAwAAAAAsBQAAAAAAADgm7gMAAAAApdGZAwAAAAAtBQAA"
+			"AAAAAEg78QMAAAAApdGZAwAAAAAuBQAAAAAAAEg78QMAAAAAj5moAwAAAAAvBQAAAAAAANEd8gMA"
+			"AAAAGHypAwAAAAAwBQAAAAAAALvlAAQAAAAAGHypAwAAAAAxBQAAAAAAAEzNAQQAAAAA9myoAwAA"
+			"AAAyBQAAAAAAAGeLAQQAAAAA7symAwAAAAAzBQAAAAAAAE+EAQQAAAAAY6+mAwAAAAA0BQAAAAAA"
+			"AOupAAQAAAAAPw+kAwAAAAA1BQAAAAAAAEmeAAQAAAAALPOjAwAAAAA2BQAAAAAAAHBd/wMAAAAA"
+			"eH2hAwAAAAA3BQAAAAAAAI9N/wMAAAAAj2OhAwAAAAA4BQAAAAAAACiu/QMAAAAAzSefAwAAAAA5"
+			"BQAAAAAAAGua/QMAAAAAsRCfAwAAAAA6BQAAAAAAAK+m+wMAAAAA9RydAwAAAAA7BQAAAAAAAJOP"
+			"+wMAAAAAOAmdAwAAAAA8BQAAAAAAANFT+QMAAAAA0WmbAwAAAAA9BQAAAAAAAOg5+QMAAAAA8Fmb"
+			"AwAAAAA+BQAAAAAAADTE9gMAAAAAFxmaAwAAAAA/BQAAAAAAACGo9gMAAAAAdQ2aAwAAAABABQAA"
+			"AAAAAP0H9AMAAAAAETOZAwAAAABBBQAAAAAAAHLq8wMAAAAA+SuZAwAAAABCBQAAAAAAAGpK8gMA"
+			"AAAAFOqYAwAAAABDBQAAAAAAAEg78QMAAAAApdGZAwAAAABEBQAAAAAAADgm7gMAAAAApdGZAwAA"
+			"AABFBQAAAAAAABYX7QMAAAAAFOqYAwAAAABGBQAAAAAAAA536wMAAAAA+SuZAwAAAABHBQAAAAAA"
+			"AINZ6wMAAAAAETOZAwAAAABIBQAAAAAAAF+56AMAAAAAdQ2aAwAAAABJBQAAAAAAAEyd6AMAAAAA"
+			"FxmaAwAAAABKBQAAAAAAAJgn5gMAAAAA8FmbAwAAAABLBQAAAAAAAK8N5gMAAAAA0WmbAwAAAABM"
+			"BQAAAAAAAO3R4wMAAAAAOAmdAwAAAABNBQAAAAAAANG64wMAAAAA9RydAwAAAABOBQAAAAAAABXH"
+			"4QMAAAAAsRCfAwAAAABPBQAAAAAAAFiz4QMAAA=="
 		)
 	)
@@
 			"DgEe9Fe2Fpz9udliOnqRHL/q4o8JP0ma4mMPUPOmFgl1xITCPP5cKl2mZd0fjje97xYft392z1fd"
 			"8y+r7pu7m8v1/LL78vq2+wNyAa7o0aZLpinKNugPvjw+Gw3GR7PN7f03yf84fXlylhTdQXLyU/L+"
-			"p/Pk3cvz4zfJycvzl2dvXr8+/x9yIKzrRN1Hau8k0dIGf1Y1+A=="
+			"p/Pk3cvz4zfJycvzl2dvXr8+/x9yIKzrRN1Hau8k0dIGf1Y1+EXrAgAAAABVCgAAAAAAACDwCAgD"
+			"AAAAwO8ICAMAAAAAAAAA/////85WXAIAAAAApErrAgAAAABWCgAAAAAAAFDwCAgDAAAA8O8ICAMA"
+			"AAAAAAAA/////2PHSgIAAAAApErrAgAAAABXCgAAAAAAAIDwCAgDAAAAIPAICAMAAAAAAAAA////"
+			"/2DHSgIAAAAApUrrAgAAAABYCgAAAAAAALDwCAgDAAAAUPAICAMAAAAAAAAA/////zllSgIAAAAA"
+			"BlbrAgAAAABZCgAAAAAAAODwCAgDAAAAgPAICAMAAAAAAAAA/////8PTSAIAAAAASgfsAgAAAABa"
+			"CgAAAAAAABDxCAgDAAAAsPAICAMAAAAAAAAA/////3KdRwIAAAAAmz3tAgAAAABbCgAAAAAAAEDx"
+			"CAgDAAAA4PAICAMAAAAAAAAA/////y7sRgIAAAAAE8/uAgAAAABcCgAAAAAAAHDxCAgDAAAAEPEI"
+			"CAMAAAAAAAAA/////8zgRgIAAAAAMjHvAgAAAABdCgAAAAAAAKDxCAgDAAAAQPEICAMAAAAAAAAA"
+			"/////8zgRgIAAAAAe0r7AgAAAABeCgAAAAAAANDxCAgDAAAAcPEICAMAAAAAAAAA//////GWRgIA"
+			"AAAAyi38AgAAAABfCgAAAAAAAADyCAgDAAAAoPEICAMAAAAAAAAA/////5XVRQIAAAAARrr8AgAA"
+			"AABgCgAAAAAAADDyCAgDAAAA0PEICAMAAAAAAAAA/////5PmRAIAAAAARrr8AgAAAABhCgAAAAAA"
+			"AGDyCAgDAAAAAPIICAMAAAAIAAAA/////zclRAIAAAAAyi38AgAAAABiCgAAAAAAAJDyCAgDAAAA"
+			"MPIICAMAAAAAAAAA/////x/gQwIAAAAA+ob7AgAAAABjCgAAAAAAAMDyCAgDAAAAYPIICAMAAAAA"
+			"AAAA//////ONQwIAAAAALoD5AgAAAABkCgAAAAAAAPDyCAgDAAAAkPIICAMAAAAAAAAA/////3Wz"
+			"QgIAAAAAt9/2AgAAAABlCgAAAAAAACDzCAgDAAAAwPIICAMAAAAAAAAA/////3NyQQIAAAAAs2n0"
+			"AgAAAABmCgAAAAAAAFDzCAgDAAAA8PIICAMAAAAAAAAA/////1rRQAIAAAAA94vzAgAAAABnCgAA"
+			"AAAAAIDzCAgDAAAAIPMICAMAAAAEAAAA/////xr1OAIAAAAANmj7AgAAAABoCgAAAAAAALDzCAgD"
+			"AAAAUPMICAMAAAAIAAAA/////2XWOAIAAAAAmvX6AgAAAABpCgAAAAAAAODzCAgDAAAAgPMICAMA"
+			"AAAAAAAA//////ruNwIAAAAAxmT5AgAAAABqCgAAAAAAABD0CA=="
 		)
 	)
@@
 			)
 		)
-		(property "LCSC" "C267415"
+		(property "LCSC" "C84703"
 			(at 229.87 121.92 0)
 			(effects
@@
 			)
 		)
-		(property "MPN" "C1005X7R222MGTS"
+		(property "MPN" "CL05B222KB5NNNC"
 			(at 229.87 121.92 0)
 			(effects
@@
 			)
 		)
-		(property "LCSC" "C267415"
+		(property "LCSC" "C84703"
 			(at 243.84 90.17 0)
 			(effects
@@
 			)
 		)
-		(property "MPN" "C1005X7R222MGTS"
+		(property "MPN" "CL05B222KB5NNNC"
 			(at 243.84 90.17 0)
 			(effects
@@
 			)
 		)
-		(property "LCSC" "C267415"
+		(property "LCSC" "C84703"
 			(at 33.02 45.72 0)
 			(effects
@@
 			)
 		)
-		(property "MPN" "C1005X7R222MGTS"
+		(property "MPN" "CL05B222KB5NNNC"
 			(at 33.02 45.72 0)
 			(effects
@@
 			)
 		)
-		(property "LCSC" "C267415"
+		(property "LCSC" "C84703"
 			(at 243.84 74.93 0)
 			(effects
@@
 			)
 		)
-		(property "MPN" "C1005X7R222MGTS"
+		(property "MPN" "CL05B222KB5NNNC"
 			(at 243.84 74.93 0)
 			(effects
@@
 			)
 		)
-		(property "LCSC" "C267415"
+		(property "LCSC" "C84703"
 			(at 229.87 90.17 0)
 			(effects
@@
 			)
 		)
-		(property "MPN" "C1005X7R222MGTS"
+		(property "MPN" "CL05B222KB5NNNC"
 			(at 229.87 90.17 0)
 			(effects
@@
 			)
 		)
-		(property "LCSC" "C267415"
+		(property "LCSC" "C84703"
 			(at 243.84 106.68 0)
 			(effects
@@
 			)
 		)
-		(property "MPN" "C1005X7R222MGTS"
+		(property "MPN" "CL05B222KB5NNNC"
 			(at 243.84 106.68 0)
 			(effects
@@
 			)
 		)
-		(property "LCSC" "C458949"
+		(property "LCSC" "C1525"
 			(at 228.6 39.37 0)
 			(effects
@@
 			)
 		)
-		(property "MPN" "MT15B104K160CT"
+		(property "MPN" "CL05B104KO5NNNC"
 			(at 228.6 39.37 0)
 			(effects
@@
 			)
 		)
-		(property "LCSC" "C267415"
+		(property "LCSC" "C84703"
 			(at 229.87 106.68 0)
 			(effects
@@
 			)
 		)
-		(property "MPN" "C1005X7R222MGTS"
+		(property "MPN" "CL05B222KB5NNNC"
 			(at 229.87 106.68 0)
 			(effects
@@
 			)
 		)
-		(property "LCSC" "C458949"
+		(property "LCSC" "C1525"
 			(at 107.95 39.37 0)
 			(effects
@@
 			)
 		)
-		(property "MPN" "MT15B104K160CT"
+		(property "MPN" "CL05B104KO5NNNC"
 			(at 107.95 39.37 0)
 			(effects
@@
 			)
 		)
-		(property "LCSC" "C267415"
+		(property "LCSC" "C84703"
 			(at 229.87 74.93 0)
 			(effects
@@
 			)
 		)
-		(property "MPN" "C1005X7R222MGTS"
+		(property "MPN" "CL05B222KB5NNNC"
 			(at 229.87 74.93 0)
 			(effects
@@
 			)
 		)
-		(property "LCSC" "C458949"
+		(property "LCSC" "C1525"
 			(at 166.37 39.37 0)
 			(effects
@@
 			)
 		)
-		(property "MPN" "MT15B104K160CT"
+		(property "MPN" "CL05B104KO5NNNC"
 			(at 166.37 39.37 0)
 			(effects
@@
 			)
 		)
-		(property "LCSC" "C267415"
+		(property "LCSC" "C84703"
 			(at 243.84 121.92 0)
 			(effects
@@
 			)
 		)
-		(property "MPN" "C1005X7R222MGTS"
+		(property "MPN" "CL05B222KB5NNNC"
 			(at 243.84 121.92 0)
 			(effects
