File: Hardware/Tatze/HoerbaerV2Tatze.kicad_pcb (KiCad board)
At the start: 2 copper layers, 80 x 84 mm, 15 parts, among them J8 PAW_A, J9 PAW_A, SW1 SW_Push, SW2 SW_Push, SW3 SW_Push, SW4 SW_Push, SW5 SW_Push

Commit message: Löcher
Parts:
- added MH10: MountingHole, MountingHole:MountingHole_2.1mm, F.Cu at (59.6, 30.8)
- added MH11: MountingHole, MountingHole:MountingHole_2.1mm, F.Cu at (112.2, 54.0)
- added MH12: MountingHole, MountingHole:MountingHole_2.1mm, F.Cu at (75.2, 84.2)
- added MH13: MountingHole, MountingHole:MountingHole_2.1mm, F.Cu at (38.1, 53.5)
- added MH5: MountingHole, MountingHole:MountingHole_2.1mm, F.Cu at (101.4, 64.0)
- added MH6: MountingHole, MountingHole:MountingHole_2.1mm, F.Cu at (86.7, 45.5)
- added MH7: MountingHole, MountingHole:MountingHole_2.1mm, F.Cu at (63.4, 45.5)
- added MH8: MountingHole, MountingHole:MountingHole_2.1mm, F.Cu at (48.6, 63.8)
- added MH9: MountingHole, MountingHole:MountingHole_2.1mm, F.Cu at (90.9, 31.0)
