File: Hardware/Tatze/HoerbaerV2Tatze.kicad_sch (KiCad schematic)
At the start: 43 parts, among them J1 SWITCH, J2 SWITCH, SW1 SW_Push, SW2 SW_Push, SW3 SW_Push, SW4 SW_Push, SW5 SW_Push, U1 74HC595, U2 74HC165

Commit message: Tatze - positions
Parts:
- removed C1, C2: C, Capacitor_SMD:C_0603_1608Metric, symbol Device:C
- removed J1, J2: SWITCH, Connector_Harwin:Harwin_M20-89006xx_1x06_P2.54mm_Horizontal, symbol Connector_Generic:Conn_01x06
- removed R1, R3, R5, R8, R9: 10k, Resistor_SMD:R_0603_1608Metric_Pad1.05x0.95mm_HandSolder, symbol Device:R
- removed R2, R4, R6, R7: R, Resistor_SMD:R_0603_1608Metric_Pad1.05x0.95mm_HandSolder, symbol Device:R
- removed TP1, TP10, TP11, TP12, TP13, TP14, TP15, TP16, TP2, TP3, TP4, TP5, TP6, TP7, TP8, TP9: TestPoint, TestPoint:TestPoint_Pad_1.5x1.5mm, symbol Connector:TestPoint
- removed U1: 74HC595, Package_SO:SOIC-16_3.9x9.9mm_P1.27mm, symbol 74xx:74HC595
- removed U2: 74HC165, Package_SO:SOIC-16_3.9x9.9mm_P1.27mm, symbol 74xx:74HC165
- added J8: PAW_A, Connector_PinHeader_2.54mm:PinHeader_2x12_P2.54mm_Vertical, symbol Connector_Generic:Conn_02x12_Odd_Even
- added J9: PAW_A, Connector_PinHeader_2.54mm:PinHeader_2x03_P2.54mm_Vertical, symbol Connector_Generic:Conn_02x03_Odd_Even
Connections:
- net GND: now also J8.10 (Pin_10), J8.14 (Pin_14), J8.18 (Pin_18), J8.2 (Pin_2), J8.22 (Pin_22), J8.6 (Pin_6), J9.4 (Pin_4); no longer D3.1 (K), D4.1 (K)
- net +9V: now reaches D1.2 (A)
- net +9V: now also D2.2 (A), D3.2 (A), D4.2 (A), J8.12 (Pin_12), J8.16 (Pin_16), J8.20 (Pin_20), J8.24 (Pin_24), J8.4 (Pin_4), J8.8 (Pin_8), J9.2 (Pin_2), J9.6 (Pin_6)
- net LED1_LOW renamed PAW_A_D1
- net PAW_A_D1: now also J8.3 (Pin_3)
- net LED2_LOW renamed PAW_A_D2
- net PAW_A_D2: now also J8.7 (Pin_7)
- net SW1 renamed PAW_A_B1
- net PAW_A_B1: now also J8.1 (Pin_1)
- net SW2 renamed PAW_A_B2
- net PAW_A_B2: now also J8.5 (Pin_5)
- net SW3 renamed PAW_A_B3
- net PAW_A_B3: now also J8.9 (Pin_9)
- net SW4 renamed PAW_A_B4
- net PAW_A_B4: now also J8.13 (Pin_13)
- net SW5 renamed PAW_A_B5
- net PAW_A_B5: now also J8.17 (Pin_17)
- new net PAW_A_B6: J8.21 (Pin_21), J9.3 (Pin_3)
- new net PAW_A_D3: D3.1 (K), J8.11 (Pin_11)
- new net PAW_A_D4: D4.1 (K), J8.15 (Pin_15)
- new net PAW_A_D5: J8.19 (Pin_19), J9.1 (Pin_1)
- new net PAW_A_D6: J8.23 (Pin_23), J9.5 (Pin_5)

Commit message: Paw
Parts:
- added MH2: MountingHole, MountingHole:MountingHole_3.2mm_M3, symbol Mechanical:MountingHole
- renumbered D4 to D1, D3 to D2, D2 to D3, D1 to D4, SW5 to SW1, SW4 to SW2, SW2 to SW4, SW1 to SW5
Connections:
- net PAW_A_B1: now also SW1.2; no longer SW5.2
- net PAW_A_B2: now also SW2.2; no longer SW4.2
- net PAW_A_B4: now also SW4.2; no longer SW2.2
- net PAW_A_B5: now also SW5.2; no longer SW1.2
- net PAW_A_D1: now also D1.1 (K); no longer D4.1 (K)
- net PAW_A_D2: now also D2.1 (K); no longer D3.1 (K)
- net PAW_A_D3: now also D3.1 (K); no longer D2.1 (K)
- net PAW_A_D4: now also D4.1 (K); no longer D1.1 (K)
Other:
- moved on the sheet: D1, D2, D3, D4, MH1, SW1, SW2, SW3, SW4

Commit message: Löcher
Parts:
- added MH10, MH11, MH12, MH13, MH5, MH6, MH7, MH8, MH9: MountingHole, MountingHole:MountingHole_2.1mm, symbol Mechanical:MountingHole
